Commit message: change in the agribot_description, Fixed the opposite coordinate, fixed the joint names difference and ready for futher operation. Further worked with ros2 parameters in both cpp and python as well

File: agribot_description/urdf/agribot.xacro (robot description, xacro)
@@ -6,7 +6,7 @@
 <link name="base_link">
   <inertial>
-    <origin xyz="0.004432349013620612 -7.841698476696025e-07 -0.004748707157977561" rpy="0 0 0"/>
+    <origin xyz="0.02376726050196793 -8.769362260032664e-06 -0.004748707157977561" rpy="0 0 0"/>
     <mass value="2.649489026530686"/>
-    <inertia ixx="0.044199" iyy="0.025957" izz="0.057874" ixy="-0.0" iyz="0.0" ixz="0.001278"/>
+    <inertia ixx="0.044199" iyy="0.025957" izz="0.057874" ixy="-0.0" iyz="-0.0" ixz="-0.001278"/>
   </inertial>
   <visual>
@@ -26,110 +26,110 @@
 <link name="motor_mount_1">
   <inertial>
-    <origin xyz="-0.0022092008966159704 -0.00456858699341936 -0.0022092008820991937" rpy="0 0 0"/>
+    <origin xyz="0.002209810412204416 0.004569033461311572 -0.002209200882099166" rpy="0 0 0"/>
+    <mass value="0.01743940222270842"/>
+    <inertia ixx="6e-06" iyy="5e-06" izz="6e-06" ixy="-1e-06" iyz="1e-06" ixz="0.0"/>
+  </inertial>
+  <visual>
+    <origin xyz="-0.333867 -0.17999 0.205668" rpy="0 0 0"/>
+    <geometry>
+      <mesh filename="file://$(find agribot_description)/meshes/motor_mount_1.stl" scale="0.001 0.001 0.001"/>
+    </geometry>
+    <material name="silver"/>
+  </visual>
+  <collision>
+    <origin xyz="-0.333867 -0.17999 0.205668" rpy="0 0 0"/>
+    <geometry>
+      <mesh filename="file://$(find agribot_description)/meshes/motor_mount_1.stl" scale="0.001 0.001 0.001"/>
+    </geometry>
+  </collision>
+</link>
+<link name="motor_mount_2">
+  <inertial>
+    <origin xyz="0.002209182927432716 0.004569033461301525 -0.002209200882099166" rpy="0 0 0"/>
+    <mass value="0.01743940222270842"/>
+    <inertia ixx="6e-06" iyy="5e-06" izz="6e-06" ixy="-1e-06" iyz="1e-06" ixz="0.0"/>
+  </inertial>
+  <visual>
+    <origin xyz="0.015838 -0.17999 0.205668" rpy="0 0 0"/>
+    <geometry>
+      <mesh filename="file://$(find agribot_description)/meshes/motor_mount_2.stl" scale="0.001 0.001 0.001"/>
+    </geometry>
+    <material name="silver"/>
+  </visual>
+  <collision>
+    <origin xyz="0.015838 -0.17999 0.205668" rpy="0 0 0"/>
+    <geometry>
+      <mesh filename="file://$(find agribot_description)/meshes/motor_mount_2.stl" scale="0.001 0.001 0.001"/>
+    </geometry>
+  </collision>
+</link>
+<link name="motor_mount_3">
+  <inertial>
+    <origin xyz="-0.002209591366516328 0.004569033461293975 -0.0022092008966213272" rpy="0 0 0"/>
+    <mass value="0.01743940222270842"/>
+    <inertia ixx="6e-06" iyy="5e-06" izz="6e-06" ixy="1e-06" iyz="1e-06" ixz="-0.0"/>
+  </inertial>
+  <visual>
+    <origin xyz="0.277468 -0.17999 0.205668" rpy="0 0 0"/>
+    <geometry>
+      <mesh filename="file://$(find agribot_description)/meshes/motor_mount_3.stl" scale="0.001 0.001 0.001"/>
+    </geometry>
+    <material name="silver"/>
+  </visual>
+  <collision>
+    <origin xyz="0.277468 -0.17999 0.205668" rpy="0 0 0"/>
+    <geometry>
+      <mesh filename="file://$(find agribot_description)/meshes/motor_mount_3.stl" scale="0.001 0.001 0.001"/>
+    </geometry>
+  </collision>
+</link>
+<link name="motor_mount_4">
+  <inertial>
+    <origin xyz="0.0022098103976929684 -0.004568140525509218 -0.002209200896621133" rpy="0 0 0"/>
+    <mass value="0.01743940222270842"/>
+    <inertia ixx="6e-06" iyy="5e-06" izz="6e-06" ixy="1e-06" iyz="-1e-06" ixz="0.0"/>
+  </inertial>
+  <visual>
+    <origin xyz="-0.333867 0.18001 0.205668" rpy="0 0 0"/>
+    <geometry>
+      <mesh filename="file://$(find agribot_description)/meshes/motor_mount_4.stl" scale="0.001 0.001 0.001"/>
+    </geometry>
+    <material name="silver"/>
+  </visual>
+  <collision>
+    <origin xyz="-0.333867 0.18001 0.205668" rpy="0 0 0"/>
+    <geometry>
+      <mesh filename="file://$(find agribot_description)/meshes/motor_mount_4.stl" scale="0.001 0.001 0.001"/>
+    </geometry>
+  </collision>
+</link>
+<link name="motor_mount_5">
+  <inertial>
+    <origin xyz="0.0022091829129214403 -0.004568140525519515 -0.002209200896621133" rpy="0 0 0"/>
+    <mass value="0.01743940222270842"/>
+    <inertia ixx="6e-06" iyy="5e-06" izz="6e-06" ixy="1e-06" iyz="-1e-06" ixz="0.0"/>
+  </inertial>
+  <visual>
+    <origin xyz="0.015838 0.18001 0.205668" rpy="0 0 0"/>
+    <geometry>
+      <mesh filename="file://$(find agribot_description)/meshes/motor_mount_5.stl" scale="0.001 0.001 0.001"/>
+    </geometry>
+    <material name="silver"/>
+  </visual>
+  <collision>
+    <origin xyz="0.015838 0.18001 0.205668" rpy="0 0 0"/>
+    <geometry>
+      <mesh filename="file://$(find agribot_description)/meshes/motor_mount_5.stl" scale="0.001 0.001 0.001"/>
+    </geometry>
+  </collision>
+</link>
+<link name="motor_mount_6">
+  <inertial>
+    <origin xyz="-0.0022095913810276646 -0.0045681405255274254 -0.0022092008820992493" rpy="0 0 0"/>
     <mass value="0.01743940222270842"/>
     <inertia ixx="6e-06" iyy="5e-06" izz="6e-06" ixy="-1e-06" iyz="-1e-06" ixz="-0.0"/>
   </inertial>
   <visual>
-    <origin xyz="0.305668 0.18 0.205668" rpy="0 0 0"/>
-    <geometry>
-      <mesh filename="file://$(find agribot_description)/meshes/motor_mount_1.stl" scale="0.001 0.001 0.001"/>
-    </geometry>
-    <material name="silver"/>
-  </visual>
-  <collision>
-    <origin xyz="0.305668 0.18 0.205668" rpy="0 0 0"/>
-    <geometry>
-      <mesh filename="file://$(find agribot_description)/meshes/motor_mount_1.stl" scale="0.001 0.001 0.001"/>
-    </geometry>
-  </collision>
-</link>
-<link name="motor_mount_2">
-  <inertial>
-    <origin xyz="-0.0022095734118441554 -0.004568586993409202 -0.0022092008820991937" rpy="0 0 0"/>
-    <mass value="0.01743940222270842"/>
-    <inertia ixx="6e-06" iyy="5e-06" izz="6e-06" ixy="-1e-06" iyz="-1e-06" ixz="-0.0"/>
-  </inertial>
-  <visual>
-    <origin xyz="-0.044038 0.18 0.205668" rpy="0 0 0"/>
-    <geometry>
-      <mesh filename="file://$(find agribot_description)/meshes/motor_mount_2.stl" scale="0.001 0.001 0.001"/>
-    </geometry>
-    <material name="silver"/>
-  </visual>
-  <collision>
-    <origin xyz="-0.044038 0.18 0.205668" rpy="0 0 0"/>
-    <geometry>
-      <mesh filename="file://$(find agribot_description)/meshes/motor_mount_2.stl" scale="0.001 0.001 0.001"/>
-    </geometry>
-  </collision>
-</link>
-<link name="motor_mount_3">
-  <inertial>
-    <origin xyz="0.0022092008821049114 -0.004568586993401569 -0.002209200896621355" rpy="0 0 0"/>
-    <mass value="0.01743940222270842"/>
-    <inertia ixx="6e-06" iyy="5e-06" izz="6e-06" ixy="1e-06" iyz="-1e-06" ixz="0.0"/>
-  </inertial>
-  <visual>
-    <origin xyz="-0.305668 0.18 0.205668" rpy="0 0 0"/>
-    <geometry>
-      <mesh filename="file://$(find agribot_description)/meshes/motor_mount_3.stl" scale="0.001 0.001 0.001"/>
-    </geometry>
-    <material name="silver"/>
-  </visual>
-  <collision>
-    <origin xyz="-0.305668 0.18 0.205668" rpy="0 0 0"/>
-    <geometry>
-      <mesh filename="file://$(find agribot_description)/meshes/motor_mount_3.stl" scale="0.001 0.001 0.001"/>
-    </geometry>
-  </collision>
-</link>
-<link name="motor_mount_4">
-  <inertial>
-    <origin xyz="-0.0022092008821046893 0.004568586993401735 -0.002209200896621133" rpy="0 0 0"/>
-    <mass value="0.01743940222270842"/>
-    <inertia ixx="6e-06" iyy="5e-06" izz="6e-06" ixy="1e-06" iyz="1e-06" ixz="-0.0"/>
-  </inertial>
-  <visual>
-    <origin xyz="0.305668 -0.18 0.205668" rpy="0 0 0"/>
-    <geometry>
-      <mesh filename="file://$(find agribot_description)/meshes/motor_mount_4.stl" scale="0.001 0.001 0.001"/>
-    </geometry>
-    <material name="silver"/>
-  </visual>
-  <collision>
-    <origin xyz="0.305668 -0.18 0.205668" rpy="0 0 0"/>
-    <geometry>
-      <mesh filename="file://$(find agribot_description)/meshes/motor_mount_4.stl" scale="0.001 0.001 0.001"/>
-    </geometry>
-  </collision>
-</link>
-<link name="motor_mount_5">
-  <inertial>
-    <origin xyz="-0.002209573397332902 0.004568586993411894 -0.002209200896621133" rpy="0 0 0"/>
-    <mass value="0.01743940222270842"/>
-    <inertia ixx="6e-06" iyy="5e-06" izz="6e-06" ixy="1e-06" iyz="1e-06" ixz="-0.0"/>
-  </inertial>
-  <visual>
-    <origin xyz="-0.044038 -0.18 0.205668" rpy="0 0 0"/>
-    <geometry>
-      <mesh filename="file://$(find agribot_description)/meshes/motor_mount_5.stl" scale="0.001 0.001 0.001"/>
-    </geometry>
-    <material name="silver"/>
-  </visual>
-  <collision>
-    <origin xyz="-0.044038 -0.18 0.205668" rpy="0 0 0"/>
-    <geometry>
-      <mesh filename="file://$(find agribot_description)/meshes/motor_mount_5.stl" scale="0.001 0.001 0.001"/>
-    </geometry>
-  </collision>
-</link>
-<link name="motor_mount_6">
-  <inertial>
-    <origin xyz="0.002209200896616137 0.00456858699341961 -0.002209200882099277" rpy="0 0 0"/>
-    <mass value="0.01743940222270842"/>
-    <inertia ixx="6e-06" iyy="5e-06" izz="6e-06" ixy="-1e-06" iyz="1e-06" ixz="0.0"/>
-  </inertial>
-  <visual>
-    <origin xyz="-0.305668 -0.18 0.205668" rpy="0 0 0"/>
+    <origin xyz="0.277468 0.18001 0.205668" rpy="0 0 0"/>
     <geometry>
       <mesh filename="file://$(find agribot_description)/meshes/motor_mount_6.stl" scale="0.001 0.001 0.001"/>
@@ -138,5 +138,5 @@
   </visual>
   <collision>
-    <origin xyz="-0.305668 -0.18 0.205668" rpy="0 0 0"/>
+    <origin xyz="0.277468 0.18001 0.205668" rpy="0 0 0"/>
     <geometry>
       <mesh filename="file://$(find agribot_description)/meshes/motor_mount_6.stl" scale="0.001 0.001 0.001"/>
@@ -146,110 +146,110 @@
 <link name="motor_1">
   <inertial>
-    <origin xyz="-0.011036049168308915 0.032900619363953165 0.010882072426481426" rpy="0 0 0"/>
+    <origin xyz="0.011036658683897693 -0.03290017289606087 0.010882072426481482" rpy="0 0 0"/>
+    <mass value="0.4814783214697331"/>
+    <inertia ixx="0.000239" iyy="7.4e-05" izz="0.000239" ixy="-1e-06" iyz="1e-06" ixz="0.0"/>
+  </inertial>
+  <visual>
+    <origin xyz="-0.338512 -0.199225 0.232233" rpy="0 0 0"/>
+    <geometry>
+      <mesh filename="file://$(find agribot_description)/meshes/motor_1.stl" scale="0.001 0.001 0.001"/>
+    </geometry>
+    <material name="silver"/>
+  </visual>
+  <collision>
+    <origin xyz="-0.338512 -0.199225 0.232233" rpy="0 0 0"/>
+    <geometry>
+      <mesh filename="file://$(find agribot_description)/meshes/motor_1.stl" scale="0.001 0.001 0.001"/>
+    </geometry>
+  </collision>
+</link>
+<link name="motor_2">
+  <inertial>
+    <origin xyz="0.011036031199125086 -0.032900172896071556 0.010882072426481482" rpy="0 0 0"/>
+    <mass value="0.4814783214697331"/>
+    <inertia ixx="0.000239" iyy="7.4e-05" izz="0.000239" ixy="-1e-06" iyz="1e-06" ixz="0.0"/>
+  </inertial>
+  <visual>
+    <origin xyz="0.011193 -0.199225 0.232233" rpy="0 0 0"/>
+    <geometry>
+      <mesh filename="file://$(find agribot_description)/meshes/motor_2.stl" scale="0.001 0.001 0.001"/>
+    </geometry>
+    <material name="silver"/>
+  </visual>
+  <collision>
+    <origin xyz="0.011193 -0.199225 0.232233" rpy="0 0 0"/>
+    <geometry>
+      <mesh filename="file://$(find agribot_description)/meshes/motor_2.stl" scale="0.001 0.001 0.001"/>
+    </geometry>
+  </collision>
+</link>
+<link name="motor_3">
+  <inertial>
+    <origin xyz="0.010881681942064958 -0.032900172896079855 -0.011036049168313078" rpy="0 0 0"/>
+    <mass value="0.4814783214697331"/>
+    <inertia ixx="0.000239" iyy="7.4e-05" izz="0.000239" ixy="1e-06" iyz="1e-06" ixz="-0.0"/>
+  </inertial>
+  <visual>
+    <origin xyz="0.304033 -0.199225 0.210313" rpy="0 0 0"/>
+    <geometry>
+      <mesh filename="file://$(find agribot_description)/meshes/motor_3.stl" scale="0.001 0.001 0.001"/>
+    </geometry>
+    <material name="silver"/>
+  </visual>
+  <collision>
+    <origin xyz="0.304033 -0.199225 0.210313" rpy="0 0 0"/>
+    <geometry>
+      <mesh filename="file://$(find agribot_description)/meshes/motor_3.stl" scale="0.001 0.001 0.001"/>
+    </geometry>
+  </collision>
+</link>
+<link name="motor_4">
+  <inertial>
+    <origin xyz="-0.011036439652719165 0.032900065831845654 0.010882072426481482" rpy="0 0 0"/>
     <mass value="0.4814783214697331"/>
     <inertia ixx="0.000239" iyy="7.4e-05" izz="0.000239" ixy="-1e-06" iyz="-1e-06" ixz="-0.0"/>
   </inertial>
   <visual>
-    <origin xyz="0.310313 0.199235 0.232233" rpy="0 0 0"/>
-    <geometry>
-      <mesh filename="file://$(find agribot_description)/meshes/motor_1.stl" scale="0.001 0.001 0.001"/>
-    </geometry>
-    <material name="silver"/>
-  </visual>
-  <collision>
-    <origin xyz="0.310313 0.199235 0.232233" rpy="0 0 0"/>
-    <geometry>
-      <mesh filename="file://$(find agribot_description)/meshes/motor_1.stl" scale="0.001 0.001 0.001"/>
-    </geometry>
-  </collision>
-</link>
-<link name="motor_2">
-  <inertial>
-    <origin xyz="-0.011036421683536465 0.032899619363963795 0.010882072426481426" rpy="0 0 0"/>
-    <mass value="0.4814783214697331"/>
-    <inertia ixx="0.000239" iyy="7.4e-05" izz="0.000239" ixy="-1e-06" iyz="-1e-06" ixz="-0.0"/>
-  </inertial>
-  <visual>
-    <origin xyz="-0.039393 0.199234 0.232233" rpy="0 0 0"/>
-    <geometry>
-      <mesh filename="file://$(find agribot_description)/meshes/motor_2.stl" scale="0.001 0.001 0.001"/>
-    </geometry>
-    <material name="silver"/>
-  </visual>
-  <collision>
-    <origin xyz="-0.039393 0.199234 0.232233" rpy="0 0 0"/>
-    <geometry>
-      <mesh filename="file://$(find agribot_description)/meshes/motor_2.stl" scale="0.001 0.001 0.001"/>
-    </geometry>
-  </collision>
-</link>
-<link name="motor_3">
-  <inertial>
-    <origin xyz="-0.010882072426476319 0.03289961936397218 -0.011036049168313106" rpy="0 0 0"/>
+    <origin xyz="0.282113 0.199244 0.232233" rpy="0 0 0"/>
+    <geometry>
+      <mesh filename="file://$(find agribot_description)/meshes/motor_4.stl" scale="0.001 0.001 0.001"/>
+    </geometry>
+    <material name="silver"/>
+  </visual>
+  <collision>
+    <origin xyz="0.282113 0.199244 0.232233" rpy="0 0 0"/>
+    <geometry>
+      <mesh filename="file://$(find agribot_description)/meshes/motor_4.stl" scale="0.001 0.001 0.001"/>
+    </geometry>
+  </collision>
+</link>
+<link name="motor_5">
+  <inertial>
+    <origin xyz="-0.010882090395659785 0.03290006583185412 -0.011036049168312329" rpy="0 0 0"/>
     <mass value="0.4814783214697331"/>
     <inertia ixx="0.000239" iyy="7.4e-05" izz="0.000239" ixy="1e-06" iyz="-1e-06" ixz="0.0"/>
   </inertial>
   <visual>
-    <origin xyz="-0.332233 0.199234 0.210313" rpy="0 0 0"/>
-    <geometry>
-      <mesh filename="file://$(find agribot_description)/meshes/motor_3.stl" scale="0.001 0.001 0.001"/>
-    </geometry>
-    <material name="silver"/>
-  </visual>
-  <collision>
-    <origin xyz="-0.332233 0.199234 0.210313" rpy="0 0 0"/>
-    <geometry>
-      <mesh filename="file://$(find agribot_description)/meshes/motor_3.stl" scale="0.001 0.001 0.001"/>
-    </geometry>
-  </collision>
-</link>
-<link name="motor_4">
-  <inertial>
-    <origin xyz="0.011036049168307749 -0.032900619363953415 0.010882072426481426" rpy="0 0 0"/>
+    <origin xyz="-0.010727 0.199244 0.210313" rpy="0 0 0"/>
+    <geometry>
+      <mesh filename="file://$(find agribot_description)/meshes/motor_5.stl" scale="0.001 0.001 0.001"/>
+    </geometry>
+    <material name="silver"/>
+  </visual>
+  <collision>
+    <origin xyz="-0.010727 0.199244 0.210313" rpy="0 0 0"/>
+    <geometry>
+      <mesh filename="file://$(find agribot_description)/meshes/motor_5.stl" scale="0.001 0.001 0.001"/>
+    </geometry>
+  </collision>
+</link>
+<link name="motor_6">
+  <inertial>
+    <origin xyz="-0.010881462910887985 0.032900065831863695 -0.011036049168313605" rpy="0 0 0"/>
     <mass value="0.4814783214697331"/>
-    <inertia ixx="0.000239" iyy="7.4e-05" izz="0.000239" ixy="-1e-06" iyz="1e-06" ixz="0.0"/>
-  </inertial>
-  <visual>
-    <origin xyz="-0.310313 -0.199235 0.232233" rpy="0 0 0"/>
-    <geometry>
-      <mesh filename="file://$(find agribot_description)/meshes/motor_4.stl" scale="0.001 0.001 0.001"/>
-    </geometry>
-    <material name="silver"/>
-  </visual>
-  <collision>
-    <origin xyz="-0.310313 -0.199235 0.232233" rpy="0 0 0"/>
-    <geometry>
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
Commit message: added base_footprint in the urdf and made changes to the rviz config so we can actually place the bot on the z=0 with wheels on contact. Also fixed the wheels rotation from <axis xyz="-0.0 -1.0 0.0"/> to <axis xyz="-0.0 1.0 0.0"/> so moves foreward when moved foreward.

File: agribot_description/urdf/agribot.xacro (robot description, xacro)
@@ -4,4 +4,5 @@
 <xacro:include filename="$(find agribot_description)/urdf/agribot.ros2control" />
 <xacro:include filename="$(find agribot_description)/urdf/agribot.gazebo" />
+<link name="base_footprint" />
 <link name="base_link">
   <inertial>
@@ -444,4 +445,9 @@
   </collision>
 </link>
+<joint name="world" type="fixed">
+  <parent link="base_footprint"/>
+  <child link="base_link"/>
+  <origin xyz="0.0 0.0 0.27431" rpy="0.0 0.0 0.0"/>
+</joint>
 <joint name="left_front_mount_joint" type="fixed">
   <origin xyz="0.333867 0.17999 -0.205668" rpy="0 0 0"/>
@@ -508,5 +514,5 @@
   <parent link="motor_4"/>
   <child link="right_rear_link_1"/>
-  <axis xyz="-0.0 -1.0 0.0"/>
+  <axis xyz="-0.0 1.0 0.0"/>
 </joint>
 <joint name="right_mid_wheel_joint" type="continuous">
@@ -514,5 +520,5 @@
   <parent link="motor_5"/>
   <child link="right_mid_link_1"/>
-  <axis xyz="0.0 -1.0 -0.0"/>
+  <axis xyz="0.0 1.0 -0.0"/>
 </joint>
 <joint name="right_front_wheel_joint" type="continuous">
@@ -520,5 +526,5 @@
   <parent link="motor_6"/>
   <child link="right_front_link_1"/>
-  <axis xyz="0.0 -1.0 -0.0"/>
+  <axis xyz="0.0 1.0 -0.0"/>
 </joint>
 <joint name="left_front_wheel_joint" type="continuous">

Commit message: agribot ros2 control setup finished now have to write the launch file for the simple controller.

File: agribot_description/urdf/agribot.xacro (robot description, xacro)
@@ -445,5 +445,5 @@
   </collision>
 </link>
-<joint name="world" type="fixed">
+<joint name="world_joint" type="fixed">
   <parent link="base_footprint"/>
   <child link="base_link"/>

Commit message: edited the collision tag for the wheels so we don't have any error.

File: agribot_description/urdf/agribot.xacro (robot description, xacro)
@@ -279,7 +279,7 @@
   </visual>
   <collision>
-    <origin xyz="0.297257 0.219744 0.226988" rpy="0 0 0"/>
-    <geometry>
-      <mesh filename="file://$(find agribot_description)/meshes/right_rear_link_1.stl" scale="0.001 0.001 0.001"/>
+    <origin xyz="0.0 -0.007 0.0" rpy="1.57 0 0"/>
+    <geometry>
+      <cylinder radius="0.05" length="0.045"/>
     </geometry>
   </collision>
@@ -299,7 +299,7 @@
   </visual>
   <collision>
-    <origin xyz="-0.004716 0.219744 0.226222" rpy="0 0 0"/>
-    <geometry>
-      <mesh filename="file://$(find agribot_description)/meshes/right_mid_link_1.stl" scale="0.001 0.001 0.001"/>
+    <origin xyz="0.0 -0.007 0.0" rpy="1.57 0 0"/>
+    <geometry>
+      <cylinder radius="0.05" length="0.045"/>
     </geometry>
   </collision>
@@ -319,7 +319,7 @@
   </visual>
   <collision>
-    <origin xyz="-0.354422 0.219744 0.226222" rpy="0 0 0"/>
-    <geometry>
-      <mesh filename="file://$(find agribot_description)/meshes/right_front_link_1.stl" scale="0.001 0.001 0.001"/>
+    <origin xyz="0.0 -0.007 0.0" rpy="1.57 0 0"/>
+    <geometry>
+      <cylinder radius="0.05" length="0.045"/>
     </geometry>
   </collision>
@@ -339,7 +339,7 @@
   </visual>
   <collision>
-    <origin xyz="-0.354422 -0.219725 0.226222" rpy="0 0 0"/>
-    <geometry>
-      <mesh filename="file://$(find agribot_description)/meshes/left_front_link_1.stl" scale="0.001 0.001 0.001"/>
+    <origin xyz="0.0 0.007 0.0" rpy="1.57 0 0"/>
+    <geometry>
+      <cylinder radius="0.05" length="0.045"/>
     </geometry>
   </collision>
@@ -359,7 +359,7 @@
   </visual>
   <collision>
-    <origin xyz="-0.004716 -0.219725 0.226222" rpy="0 0 0"/>
-    <geometry>
-      <mesh filename="file://$(find agribot_description)/meshes/left_mid_link_1.stl" scale="0.001 0.001 0.001"/>
+    <origin xyz="0.0 0.007 0.0" rpy="1.57 0 0"/>
+    <geometry>
+      <cylinder radius="0.05" length="0.045"/>
     </geometry>
   </collision>
@@ -379,7 +379,7 @@
   </visual>
   <collision>
-    <origin xyz="0.298023 -0.219725 0.226222" rpy="0 0 0"/>
-    <geometry>
-      <mesh filename="file://$(find agribot_description)/meshes/left_rear_link_1.stl" scale="0.001 0.001 0.001"/>
+    <origin xyz="0.0 0.007 0.0" rpy="1.57 0 0"/>
+    <geometry>
+      <cylinder radius="0.05" length="0.045"/>
     </geometry>
   </collision>
