Commit message: added imu sensor in agribot.gazebo

File: src/agribot_description/urdf/agribot.xacro (robot description, xacro)
@@ -385,5 +385,5 @@
   </collision>
 </link>
-<link name="imu_link_1">
+<link name="imu_link">
   <inertial>
     <origin xyz="0.0001505183280713085 0.0009028305958420219 -0.0007671413731985752" rpy="0 0 0"/>
@@ -549,5 +549,5 @@
   <origin xyz="0.0782 0.09499 0.028" rpy="0 0 0"/>
   <parent link="base_link"/>
-  <child link="imu_link_1"/>
+  <child link="imu_link"/>
 </joint>
 <joint name="lidar_joint" type="fixed">

Commit message: fixed the manual bug i created

File: src/agribot_description/urdf/agribot.xacro (robot description, xacro)
@@ -385,5 +385,5 @@
   </collision>
 </link>
-<link name="imu_link">
+<link name="imu_link_1">
   <inertial>
     <origin xyz="0.0001505183280713085 0.0009028305958420219 -0.0007671413731985752" rpy="0 0 0"/>
@@ -549,5 +549,5 @@
   <origin xyz="0.0782 0.09499 0.028" rpy="0 0 0"/>
   <parent link="base_link"/>
-  <child link="imu_link"/>
+  <child link="imu_link_1"/>
 </joint>
 <joint name="lidar_joint" type="fixed">
